File: Raspberry_Pi_Hat.sch (KiCad schematic (older format))
At the start: 9 parts, among them J1 Raspberry_Pi_2_3, SW1 SW_DPST, U1 DHT22

Commit message: routes board, gerber files and BOM
Parts:
- J1: footprint Connector_PinSocket_2.54mm:PinSocket_2x08_P2.54mm_Vertical -> Connector_PinHeader_2.54mm:PinHeader_2x08_P2.54mm_Vertical
- R1, R4: value R -> 10kΩ
- R2, R3: value R -> 330Ω
- U1: footprint Connector_PinHeader_2.54mm:PinHeader_1x03_P2.54mm_Vertical -> Connector_PinHeader_2.54mm:PinHeader_1x04_P2.54mm_Vertical
Changed lines of the file:
@@
 F 0 "J1" H 6750 5200 50  0000 C CNN
 F 1 "Raspberry_Pi_2_3" H 6700 5150 50  0000 C CNN
-F 2 "Connector_PinSocket_2.54mm:PinSocket_2x08_P2.54mm_Vertical" H 6100 3850 50  0001 C CNN
+F 2 "Connector_PinHeader_2.54mm:PinHeader_2x08_P2.54mm_Vertical" H 6100 3850 50  0001 C CNN
 F 3 "https://www.raspberrypi.org/documentation/hardware/raspberrypi/schematics/rpi_SCH_3bplus_1p0_reduced.pdf" H 6100 3850 50  0001 C CNN
 	1    6100 3850
@@
 P 7400 3750
 F 0 "R3" H 7470 3796 50  0000 L CNN
-F 1 "R" H 7470 3705 50  0000 L CNN
+F 1 "330Ω" H 7470 3705 50  0000 L CNN
 F 2 "Resistor_SMD:R_0805_2012Metric" V 7330 3750 50  0001 C CNN
 F 3 "~" H 7400 3750 50  0001 C CNN
@@
 P 3100 3400
 F 0 "R1" H 3170 3446 50  0000 L CNN
-F 1 "R" H 3170 3355 50  0000 L CNN
+F 1 "10kΩ" H 3170 3355 50  0000 L CNN
 F 2 "Resistor_SMD:R_0805_2012Metric" V 3030 3400 50  0001 C CNN
 F 3 "~" H 3100 3400 50  0001 C CNN
@@
 F 0 "U1" H 4106 3996 50  0000 R CNN
 F 1 "DHT22" H 4106 3905 50  0000 R CNN
-F 2 "Connector_PinHeader_2.54mm:PinHeader_1x03_P2.54mm_Vertical" H 4106 3859 50  0001 R CNN
+F 2 "Connector_PinHeader_2.54mm:PinHeader_1x04_P2.54mm_Vertical" H 4106 3859 50  0001 R CNN
 F 3 "http://akizukidenshi.com/download/ds/aosong/DHT11.pdf" H 4500 4200 50  0001 C CNN
 	1    4350 3950
@@
 P 4650 3350
 F 0 "R2" V 4443 3350 50  0000 C CNN
-F 1 "R" V 4534 3350 50  0000 C CNN
+F 1 "330Ω" V 4534 3350 50  0000 C CNN
 F 2 "Resistor_SMD:R_0805_2012Metric" V 4580 3350 50  0001 C CNN
 F 3 "~" H 4650 3350 50  0001 C CNN
@@
 P 8050 3750
 F 0 "R4" H 8120 3796 50  0000 L CNN
-F 1 "R" H 8120 3705 50  0000 L CNN
+F 1 "10kΩ" H 8120 3705 50  0000 L CNN
 F 2 "Resistor_SMD:R_0805_2012Metric" V 7980 3750 50  0001 C CNN
 F 3 "~" H 8050 3750 50  0001 C CNN
